File: PCB_SLAVE.sch (KiCad schematic (older format))
At the start: 44 parts, among them J1 RGB, J10 DHT, J2 POWER_12V, J3 MOTOR_DC, J4 LED_OUT, J7 MOTOR, J8 zigbee, J9 DAT, K1 G5LE-1, Q1 2SC1815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

Commit message: edit
Connections:
- net +5V: no longer J8.1 (Pin_1)
- net +3V3: now reaches A1.17 (3V3)
- net +3V3: now also J8.1 (Pin_1)
Changed lines of the file:
@@
-$EndComp
-$Comp
-L power:+5V #PWR019
-U 1 1 5FB7DB02
-P 8600 750
-F 0 "#PWR019" H 8600 600 50  0001 C CNN
-F 1 "+5V" V 8615 878 50  0000 L CNN
-F 2 "" H 8600 750 50  0001 C CNN
-F 3 "" H 8600 750 50  0001 C CNN
-	1    8600 750
-	0    -1   -1   0
 $EndComp
 $Comp
@@
 	-1   0    0    1
 $EndComp
+$Comp
+L power:+3.3V #PWR?
+U 1 1 5FDD6459
+P 5150 1000
+F 0 "#PWR?" H 5150 850 50  0001 C CNN
+F 1 "+3.3V" H 5165 1173 50  0000 C CNN
+F 2 "" H 5150 1000 50  0001 C CNN
+F 3 "" H 5150 1000 50  0001 C CNN
+	1    5150 1000
+	1    0    0    -1
+$EndComp
+Wire Wire Line
+	5150 1000 5150 1050
+$Comp
+L power:+3.3V #PWR?
+U 1 1 5FDDE1E2
+P 8600 750
+F 0 "#PWR?" H 8600 600 50  0001 C CNN
+F 1 "+3.3V" V 8615 878 50  0000 L CNN
+F 2 "" H 8600 750 50  0001 C CNN
+F 3 "" H 8600 750 50  0001 C CNN
+	1    8600 750
+	0    -1   -1   0
+$EndComp
 $EndSCHEMATC
