File: PCB_SLAVE.sch (KiCad schematic (older format))
At the start: 44 parts, among them J1 RGB, J10 DHT, J2 POWER_12V, J3 MOTOR_DC, J4 LED_OUT, J7 MOTOR, J8 zigbee, J9 DAT, K1 G5LE-1, Q1 2SC1815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

Commit message: edit
Parts:
- removed D2: LED_Small, Connector_PinHeader_2.54mm:PinHeader_1x02_P2.54mm_Vertical, symbol Device:LED_Small
- removed R11: 1K, Resistor_THT:R_Axial_DIN0207_L6.3mm_D2.5mm_P10.16mm_Horizontal, symbol Device:R_Small
- added C? (x2): 100nF, Capacitor_THT:CP_Radial_D5.0mm_P2.50mm, symbol Device:C_Small
- added C?: 104, Capacitor_THT:CP_Radial_D5.0mm_P2.50mm, symbol Device:C_Small
- added D?: LED_Nguon, LED_THT:LED_D3.0mm, symbol Device:LED_Small
- added Q?: 2SC1815, symbol Device:Q_NPN_BCE
- added R?: 1K, Resistor_THT:R_Axial_DIN0309_L9.0mm_D3.2mm_P15.24mm_Horizontal, symbol Device:R_Small
- added R?: 470, Resistor_THT:R_Axial_DIN0309_L9.0mm_D3.2mm_P15.24mm_Horizontal, symbol Device:R_Small
- C3: value 100nF -> 104
- C4: value 2200uF -> 1000uF
- D1: value 1N4001 -> 1N4148
- D3: value LED_Small -> LED_PHUN
- D4, D7: value 1N4008 -> 1N4148
- J2: value POWER_12V -> POWER _ 12V
- J4: value LED_OUT -> LED_TUOI
- R3: value 330 -> 220
- R6: value 1K -> 470
- R8: value 330 -> 1K
- SW2: value SW_Push -> CLEAR_EPR
- SW3: value SW_Push -> RST
Connections:
- net +12V: now also D?.2 (A), R?.1
- net +5V: now also C5.1, C?.1, C?.2
- net GND: now also SW2.1, C?.1, C?.2, C?.2, Q?.3 (E); no longer SW2.2
- net at D7.1 (K), J3.1 (Pin_1), K1.1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: now also C?.1; no longer C5.1
- net CLEAR_EPR: no longer names the net of A1.5 (D2)
- net CLEAR_EPR: now also SW2.2; no longer SW2.1
- new net: Q?.1 (B), R?.2
- new net: Q?.2 (C), R?.2
- new net: D?.1 (K), R?.1
Other:
- note added: "LED_NGUON\n"
- note added: "MOTOR_DC\n"
- note added: "POWER\n"
- note removed: "CLEAR_EPROM"
- note removed: "CONTROL_MOTOR"
- note removed: "POWER_SWITCH\n"
- moved on the sheet: A1, BZ1, C1, C2, C3, C4, C5, D1, D3, D4, D5, D6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

Commit message: add file
Parts:
- removed D6: LED_Small, LED_THT:LED_D3.0mm, symbol Device:LED_Small
- removed R12: 330, Resistor_THT:R_Axial_DIN0309_L9.0mm_D3.2mm_P15.24mm_Horizontal, symbol Device:R_Small
- added C9: 104, Capacitor_THT:C_Disc_D3.0mm_W1.6mm_P2.50mm, symbol Device:C_Small
- added R14: 10R, Resistor_THT:R_Axial_DIN0309_L9.0mm_D3.2mm_P15.24mm_Horizontal, symbol Device:R_Small
- C2: footprint Capacitor_THT:CP_Radial_D5.0mm_P2.50mm -> Capacitor_THT:CP_Radial_D5.0mm_P2.00mm
- C3: footprint Capacitor_THT:CP_Radial_D5.0mm_P2.50mm -> Capacitor_THT:C_Disc_D3.0mm_W1.6mm_P2.50mm
- C5: value 100nF -> 104; footprint Capacitor_THT:CP_Radial_D5.0mm_P2.50mm -> Capacitor_THT:C_Disc_D3.0mm_W1.6mm_P2.50mm
- C6: renamed from C?; footprint Capacitor_THT:CP_Radial_D5.0mm_P2.50mm -> Capacitor_THT:C_Disc_D3.0mm_W1.6mm_P2.50mm
- C7, C8: renamed from C?; value 100nF -> 104; footprint Capacitor_THT:CP_Radial_D5.0mm_P2.50mm -> Capacitor_THT:C_Disc_D3.0mm_W1.6mm_P2.50mm
- J1: footprint Connector_PinHeader_2.54mm:PinHeader_1x04_P2.54mm_Vertical -> Connector_PinHeader_1.00mm:PinHeader_1x04_P1.00mm_Vertical
- Q1, Q3: footprint Package_TO_SOT_THT:TO-92_Inline -> Connector_PinHeader_1.27mm:PinHeader_1x03_P1.27mm_Vertical
- Q4: renamed from Q?; footprint (none) -> Connector_PinHeader_1.27mm:PinHeader_1x03_P1.27mm_Vertical
- gave numbers to parts that had none: 3
Connections:
- net +5V: now also C9.2, R14.2; no longer BZ1.1 (-), C5.1, C7.1, C8.2, J10.1 (Pin_1), J8.1 (Pin_1), J9.4 (Pin_4)
- net GND: now also C9.1
- net ZIG_RX: now also A1.7 (D4); no longer A1.6 (D3)
- net ZIG_TX: now also A1.6 (D3); no longer A1.7 (D4)
- net +3V3: now reaches A1.17 (3V3)
- net +3V3: now also C5.1, C7.1, C8.2, J10.1 (Pin_1), J8.1 (Pin_1), J9.4 (Pin_4)
- new net: BZ1.1 (-), R14.1
Other:
- moved on the sheet: BZ1, Q3, R8

Commit message: add file
Connections:
- net +3V3: no longer C8.2, J9.4 (Pin_4)
- net +5V: now also C8.2, J9.4 (Pin_4)
Changed lines of the file:
@@
-$EndComp
-$Comp
-L power:+3.3V #PWR026
-U 1 1 5FE19778
-P 8700 3675
-F 0 "#PWR026" H 8700 3525 50  0001 C CNN
-F 1 "+3.3V" V 8715 3803 50  0000 L CNN
-F 2 "" H 8700 3675 50  0001 C CNN
-F 3 "" H 8700 3675 50  0001 C CNN
-	1    8700 3675
-	0    -1   -1   0
 $EndComp
 $Comp
@@
 	0    -1   -1   0
 $EndComp
+$Comp
+L power:+5V #PWR?
+U 1 1 5FEA2488
+P 8700 3675
+F 0 "#PWR?" H 8700 3525 50  0001 C CNN
+F 1 "+5V" V 8715 3803 50  0000 L CNN
+F 2 "" H 8700 3675 50  0001 C CNN
+F 3 "" H 8700 3675 50  0001 C CNN
+	1    8700 3675
+	0    -1   -1   0
+$EndComp
